Commit message: fix fast loop policy

File: m0609.white.urdf (robot description, URDF)
Before this commit: robot m0609, 8 links, 7 joints
Joints:
- joint joint_1: origin xyz=0 0 0.1525 rpy=0 0 0 -> xyz=0 0 0.1345 rpy=0 0 0
- joint joint_2: origin xyz=0 0.006 0 rpy=0 -1.571 -1.571 -> xyz=0 0.0062 0 rpy=0 -1.571 -1.571
